File: hard/DigiCar.brd (EAGLE design)
At the start: 68.6 x 48.3 mm, 41 parts, among them CN1 EH-2, CN11 ZX62-B-5PA(11), CN2 EH-2, CN3 EH-2, Q1 2SC2712, Q2 2SC2712, SW1 SS-12SDP2, SW2 SKRPACE010, U1 TC1262-3.3VDB, U2 DRV8835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

Commit message: READMEとCADデータを修正
Parts:
- moved C6 246.1 mm to (73.3, 46.0)
- moved C7 246.1 mm to (73.3, 42.2)
- moved R3 246.1 mm to (73.3, 27.0)
- moved R4 246.1 mm to (73.3, 23.2)
- moved R5 246.1 mm to (73.3, 19.4)
- moved R6 246.1 mm to (73.3, 15.6)
- moved R7 246.1 mm to (73.3, 11.7)
- moved R8 246.1 mm to (73.3, 7.94)
- moved C8 246.1 mm to (73.3, 38.4)
- moved R1 246.1 mm to (73.3, 34.6)
- moved R2 246.1 mm to (73.3, 30.8)
- moved CN10 199.1 mm to (56.2, 15.2)
- moved CN12 199.1 mm to (58.4, 8.89)
- moved CN5 199.1 mm to (56.2, 40.6)
- moved CN6 199.1 mm to (56.2, 35.6)
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Routing:
- net +3V3: track 103.9 -> 0.00 mm, vias 1 -> 0
- net TOF_SHDN0: track 72.0 -> 0.00 mm, vias 2 -> 0
- net BOOT: track 61.5 -> 0.00 mm, vias 3 -> 0
- net SDA: track 55.8 -> 0.00 mm, vias 3 -> 0
- net TOF_SHDN1: track 54.9 -> 0.00 mm, vias 1 -> 0
- net TOF_SHDN2: track 53.5 -> 0.00 mm, vias 1 -> 0
- net SCL: track 52.1 -> 0.00 mm, vias 3 -> 0
- net SERVO_PWM: track 46.8 -> 0.00 mm, vias 2 -> 0
- net IO19_MISO: track 45.6 -> 0.00 mm, vias 2 -> 0
- net IO18_SCK: track 44.6 -> 0.00 mm, vias 2 -> 0
- net IO5_SS: track 43.8 -> 0.00 mm, vias 2 -> 0
- net MOTOR_B_IN2: track 43.5 -> 0.00 mm, vias 2 -> 0
- net BATT_CHECK: track 41.7 -> 0.00 mm, vias 2 -> 0
- net MOTOR_B_IN1: track 41.5 -> 0.00 mm, vias 2 -> 0
- net MOTOR_A_IN1: track 40.2 -> 0.00 mm, vias 2 -> 0
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- removed copper zone on layer 1, net +3V3
- removed copper zone on layer 1, net A01
- removed copper zone on layer 1, net A02
- removed copper zone on layer 1, net A06
- removed copper zone on layer 1, net A07
- removed copper zone on layer 1, net GND
- removed copper zone on layer 16, net GND
- removed copper zone on layer 16, net N$10
- removed copper zone on layer 16, net N$11
- removed copper zone on layer 1, net N$2
- removed copper zone on layer 16, net N$28
- removed copper zone on layer 16, net N$30
- removed copper zone on layer 1, net N$31
- removed copper zone on layer 1, net N$32
- removed copper zone on layer 1, net N$34
- removed copper zone on layer 1, net N$4
- removed copper zone on layer 1, net N$5
- removed copper zone on layer 1, net N$6
- removed copper zone on layer 16, net N$9
- removed copper zone on layer 1, net V_BATT
Other:
- board outline removed
- board text removed: "+"
- board text removed: "-"
- board text removed: "0"
- board text removed: "1"
- board text removed: "17"
- board text removed: "18"
- board text removed: "2"
- board text removed: "A2 A1 A0"
- board text removed: "B"
- board text removed: "BOOT"
- board text removed: "GPduino-T"
- board text removed: "L"
- board text removed: "R"
- board text removed: "T"

Commit message: 回路を修正
Parts:
- added LED3: RED, lipoyang_discrete:LED1608
- added R9: 1k, lipoyang_cr:CP1608
Connections:
- new net N$2: LED3.A, R9.SMD2
- net GND: now also LED3.C
- net IO2: now also R9.SMD1
Changed lines of the file:
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@@
 <element name="R7" library="lipoyang_cr" package="CP1608" value="1k" x="73.3425" y="11.7475"/>
 <element name="R8" library="lipoyang_cr" package="CP1608" value="1k" x="73.3425" y="7.9375"/>
+<element name="R9" library="lipoyang_cr" package="CP1608" value="1k" x="4.7625" y="10.16"/>
+<element name="LED3" library="lipoyang_discrete" package="LED1608" value="RED" x="4.445" y="2.8575"/>
 </elements>
 <signals>
@@
 <contactref element="C8" pad="SMD2"/>
 <contactref element="R2" pad="SMD1"/>
+<contactref element="LED3" pad="C"/>
 <wire x1="81.28" y1="35.3187" x2="90.805" y2="36.195" width="0" layer="19" extent="1-1"/>
 <wire x1="81.28" y1="41.5165" x2="81.28" y2="35.3187" width="0" layer="19" extent="1-1"/>
@@
 <wire x1="34.2925" y1="3.83" x2="35.2425" y2="5.08" width="0" layer="19" extent="1-1"/>
 <wire x1="37.8125" y1="50.879" x2="52.3875" y2="40.64" width="0" layer="19" extent="1-1"/>
+<wire x1="3.695" y1="2.8575" x2="13.97" y2="2.54" width="0" layer="19" extent="1-1"/>
 </signal>
 <signal name="V_BATT">
@@
 <contactref element="U3" pad="24"/>
 <contactref element="CN12" pad="13"/>
+<contactref element="R9" pad="SMD1"/>
 <wire x1="25.855" y1="40.02" x2="64.77" y2="7.62" width="0" layer="19" extent="1-1"/>
+<wire x1="3.9125" y1="10.16" x2="25.855" y2="40.02" width="0" layer="19" extent="1-1"/>
+</signal>
+<signal name="N$2">
+<contactref element="R9" pad="SMD2"/>
+<contactref element="LED3" pad="A"/>
+<wire x1="5.6125" y1="10.16" x2="5.195" y2="2.8575" width="0" layer="19" extent="1-1"/>
 </signal>
 </signals>

Commit message: ボードに基板外形を作図
Parts:
- moved C3 47.6 mm to (80.6, 67.0)
- moved C7 47.6 mm to (73.3, 89.9)
- moved C8 47.6 mm to (73.3, 86.0)
- moved CN11 47.6 mm to (36.5, 95.9)
- moved CN8 47.6 mm to (56.2, 73.0)
- moved R5 47.6 mm to (73.3, 67.0)
- moved U1 47.6 mm to (81.3, 86.0)
- moved U3 47.6 mm to (14.6, 81.9)
- moved C1 47.6 mm to (80.6, 62.2)
- moved C2 47.6 mm to (79.7, 71.4)
- moved C5 47.6 mm to (40.0, 72.7)
- moved CN10 47.6 mm to (56.2, 62.9)
- moved CN12 47.6 mm to (58.4, 56.5)
- moved CN2 47.6 mm to (42.5, 83.5)
- moved CN4 47.6 mm to (82.2, 53.0)
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Other:
- board outline added: 164 x 42 mm
