File: hard/DigiCar.brd (EAGLE design)
At the start: 164 x 42 mm, 43 parts, among them CN1 EH-2, CN11 ZX62-B-5PA(11), CN2 EH-2, CN3 EH-2, Q1 2SC2712, Q2 2SC2712, SW1 SS-12SDP2, SW2 SKRPACE010, U1 TC1262-3.3VDB, U2 DRV8835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

Commit message: ToFセンサを配置(仮)
Parts:
- moved CN8 122.7 mm to (157.0, 3.00), turned to 30 degrees
- moved CN9 116.7 mm to (163.0, 21.0), turned to 90 degrees
- moved CN10 103.6 mm to (157.0, 39.0), turned to 150 degrees
- moved CN5 98.4 mm to (7.00, 3.00), turned to 330 degrees
- moved CN6 83.1 mm to (1.00, 21.0), turned to 270 degrees
- moved CN7 62.8 mm to (7.00, 39.0), turned to 210 degrees
